File: pcb-guide-sim.kicad_sch (KiCad schematic)
At the start: 0 parts

Commit message: Adjust page settings
Other:
- title: (none) -> PCB Guide: Simulation of Reverse Polarity Protection
Changed lines of the file:
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@@
 	(generator "eeschema")
 	(generator_version "10.0")
-	(paper "A4")
+	(paper "USLetter")
+	(title_block
+		(title "PCB Guide: Simulation of Reverse Polarity Protection")
+		(date "2026-07-07")
+		(rev "1")
+	)
 	(sheet_instances
 		(path "/"
@@
 	)
 	(embedded_fonts no)
+	(embedded_files
+		(file
+			(name "Simple Sheet.kicad_wks")
+			(type worksheet)
+			(data |KLUv/WATB8UQAPbYTiAQtRtqMSSdbV9NZNpN0B9pcXyfWiIhknMYYEUEQDBwOEcAPwBFAHd+mM+4
+				V6iairz5joK8Uq9QUc0+ouGH/AkAQEAAet7DSCkmzEQ7x3jgxNf+vF5dU1B0t0FGydXS8PqHAAgI
+				wg4I002OdggBPx30e71ey73HkePU4ay3sXtPn33z3FWPvZMn/urfZznJkrvqVXPs5r/zw2li/2Z9
+				zu9n/+0G2t9o6I3NlWoCsbupAycUpUuzGpjLkmUYacAM/9m494quf3WORRn6oYdTSW5LJCuO27bF
+				NhAAX22muZIcWnDqiT/kv30VDZXkWIlCl6s0AUEBIeXi8NAsinZdj+zdNwaqO2JJLgjmoA6OevMp
+				J6jEBdEwzXuqLRYT//yuzfB1cFIWsSsXxaKMaNZ5duODlEywDLtclY9XOF6g8UClIBoSKUiSFDpw
+				RMQGqw4QBsKHeJ55AQhE3gjPYXAvikUgvEa5VoYB0zP8l8HLhfajucwOF54EeWmE4woLl5L+IARH
+				4JkXFtoEotfEQH5g/9U/BzGsRInszOyBel7DOA018UNDSZudPOyVS/RqAR211QwBQrSHlBeFCr13
+				AB/0/pj3wRoBmSIs0brj33tp2rSOT5s48DnUk9IDn5pwIQ8Mcq1D4pSHl63ogfrV4XCAI3IZ6TIn
+				JTfpLcvLZSLBTvyOvUavpjppF279E46HqJ+MNCAdg1cF|
+			)
+			(checksum "86415F3213CB9B4651533CCE06D6A73F")
+		)
+	)
 )

Commit message: Create a simple schematic to simulate
Parts:
- added R1: 10k, symbol Device:R
- added V1: VPULSE, symbol Simulation_SPICE:VPULSE
Connections:
- new net: R1.1, V1.1
- new net GND: R1.2, V1.2
